File: LED.kicad_sch (KiCad schematic)
At the start: 15 parts, among them J35 LED 1, J36 LED 2, Q1 IRLZ44N, Q2 IRLZ44N, Q3 IRLZ44N, U4 TC4427CPA, U5 TC4427CPA

Commit message: updated 1.0
Changed lines of the file:
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@@
+		)
+	)
+	(label "12V_LED_FUSED"
+		(at 228.6 71.12 0)
+		(effects
+			(font
+				(size 1.27 1.27)
+			)
+			(justify left bottom)
+		)
+	)
+	(label "12V_LED_FUSED"
+		(at 231.14 106.68 0)
+		(effects
+			(font
+				(size 1.27 1.27)
+			)
+			(justify left bottom)
 		)
 	)
