File: PCB_Test.kicad_pcb (KiCad board)
At the start: 4 copper layers, 233.1 x 109.2 mm, 72 parts, among them J1 Peltier, J10 Raspberry Pi 5, J13 3V3 I2C, J15 3V3 I2C, J17 3V3 I2C, J18 5V I2C, J19 3V3 I2C, J2 FAN 1, J20 Switch_2, J21 Camera, J22 DS12B20, J23 DS12B20, J24 DS12B20, J25 DS12B20, J26 DHT22, J27 DHT22, J3 FAN 2, J33 left, J34 right, J35 LED 1, J36 LED 2, J4 FAN 3, J5 Switch_1, J6 FAN 4, J7 PCIe Header, J8 4 Pin Molex Header, J9 5V I2C, Q1 IRLZ44N, Q2 IRLZ44N, Q3 IRLZ44N, U1 ESP32-DEVKITC-32E, U2 TC4427CPA, U3 TC4427CPA, U4 TC4427CPA, U5 TC4427CPA

Commit message: updated 1.0
Parts:
- added H1: MountingHole, MountingHole:MountingHole_4mm_Pad, F.Cu at (37.0, 52.0)
- added H2: MountingHole, MountingHole:MountingHole_4mm_Pad, F.Cu at (244.0, 52.0)
- added H3: MountingHole, MountingHole:MountingHole_4mm_Pad, F.Cu at (37.0, 146.0)
- added H4: MountingHole, MountingHole:MountingHole_4mm_Pad, F.Cu at (244.0, 146.0)
- added J11: Peltier, TerminalBlock:TerminalBlock_Xinya_XY308-2.54-2P_1x02_P2.54mm_Horizontal, F.Cu at (239.3, 130.0)
- added R27: 10k, Resistor_THT:R_Axial_DIN0207_L6.3mm_D2.5mm_P10.16mm_Horizontal, F.Cu at (231.1, 121.3)
- F3: value Fuse 15A -> Fuse 30A
- J8: footprint Footprint:231834001000 -> Footprint:4_pin_Molex
- moved J20 155.2 mm to (173.4, 73.3)
- moved R25 154.8 mm to (189.1, 70.1), turned to 0 degrees
- moved R26 153.9 mm to (184.3, 70.4)
- moved R24 117.6 mm to (162.0, 71.2), turned to 180 degrees
- moved R23 108.3 mm to (147.8, 81.5)
- moved J5 107.6 mm to (138.3, 73.5)
- moved J8 27.5 mm to (222.4, 53.2)
- moved J21 26.3 mm to (57.1, 97.2)
- moved J10 13.3 mm to (43.3, 68.0)
- moved J1 13.0 mm to (236.3, 146.6)
- moved C6 12.5 mm to (210.9, 106.3)
- moved C5 12.5 mm to (223.3, 107.3)
- moved C7 12.5 mm to (227.1, 79.8)
- moved C8 12.5 mm to (227.6, 66.8)
- moved D1 12.5 mm to (199.8, 106.2)
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Connections:
- C5 pad 1: +12V -> /Power Distribution/12V_FUSED_MAIN
- C6 pad 1: +12V -> /Power Distribution/12V_FUSED_MAIN
- D1 pad 2: +12V -> /Power Distribution/12V_FUSED_MAIN
- F3 pad 2: Net-(J7-POWER_1) -> /Power Distribution/12V_FUSED_MAIN
- J7 pad 10: +12V -> /Power Distribution/12V_FUSED_MAIN
- J7 pad 5: Net-(J7-POWER_1) -> /Power Distribution/12V_FUSED_MAIN
- J7 pad 6: Net-(J7-POWER_1) -> /Power Distribution/12V_FUSED_MAIN
- J7 pad 7: Net-(J7-POWER_1) -> /Power Distribution/12V_FUSED_MAIN
- J7 pad 8: Net-(J7-POWER_1) -> /Power Distribution/12V_FUSED_MAIN
- J7 pad 9: +12V -> /Power Distribution/12V_FUSED_MAIN
Routing:
- added copper zone on In1.Cu, net GND
Other:
- board size 233.1 x 109.2 mm -> 221 x 109.2 mm

Commit message: Describe the task you completed
Parts:
- moved D1 18.5 mm to (187.9, 92.0), turned to 0 degrees
- moved C5 15.6 mm to (210.2, 98.8), turned to -90 degrees
- moved C6 8.85 mm to (203.5, 101.5), turned to 180 degrees
- moved F3 7.80 mm to (212.1, 92.0), turned to 0 degrees
- moved F4 6.05 mm to (215.9, 73.8)
- moved C7 3.74 mm to (228.2, 76.2)
- moved C8 3.74 mm to (228.8, 63.2)
- moved J21 2.67 mm to (58.2, 99.6)
Connections:
- C5 pad 1: /Power Distribution/12V_FUSED_MAIN -> +12V
- C6 pad 1: /Power Distribution/12V_FUSED_MAIN -> +12V
- D1 pad 2: /Power Distribution/12V_FUSED_MAIN -> +12V
Routing:
- net GPIO 5: track 0.00 -> 100.0 mm, vias 0 -> 2
- net GPIO 7: track 0.00 -> 82.1 mm, vias 0 -> 2
- net GPIO 24: track 0.00 -> 81.9 mm
- net GPIO 10: track 0.00 -> 53.0 mm, vias 0 -> 2
- net GPIO 11: track 0.00 -> 51.4 mm
- net GPIO 23: track 0.00 -> 47.6 mm, vias 0 -> 2
- net Net-(Q1-G): track 0.00 -> 39.4 mm
- net +5V: track 0.00 -> 38.8 mm
- net Net-(Q3-G): track 0.00 -> 37.8 mm
- net GPIO 2: track 0.00 -> 36.4 mm
- net Net-(Q2-G): track 0.00 -> 32.2 mm, vias 0 -> 2
- net GPIO 9: track 0.00 -> 21.1 mm, vias 0 -> 2
- net GPIO 3: track 0.00 -> 19.4 mm, vias 0 -> 2
- added copper zone on F.Cu, net +12V
- added copper zone on B.Cu, net /Power Distribution/12V_FUSED_MAIN
- added copper zone on F.Cu, net /Power Distribution/12V_FUSED_MAIN

Commit message: version 1.0
Parts:
- removed H1, H2, H3, H4: MountingHole, MountingHole:MountingHole_4mm_Pad
- added FID1: Fiducial, Fiducial:Fiducial_0.75mm_Mask1.5mm, F.Cu at (32.3, 58.2)
- added FID2: Fiducial, Fiducial:Fiducial_0.75mm_Mask1.5mm, F.Cu at (248.5, 58.1)
- added FID3: Fiducial, Fiducial:Fiducial_0.75mm_Mask1.5mm, F.Cu at (32.9, 140.2)
- added FID4: Fiducial, Fiducial:Fiducial_0.75mm_Mask1.5mm, F.Cu at (248.4, 140.3)
- added G***: LOGO, LOGO, F.Cu at (192.5, 51.9)
- F4: value Fuse 2A -> Fuse 11A; footprint Fuse:Fuse_Blade_ATO_directSolder -> Fuse:Fuseholder_Cylinder-5x20mm_Schurter_0031_8201_Horizontal_Open
- J11: footprint TerminalBlock:TerminalBlock_Xinya_XY308-2.54-2P_1x02_P2.54mm_Horizontal -> TerminalBlock:TerminalBlock_MaiXu_MX126-5.0-02P_1x02_P5.00mm
- J13, J17, J9: footprint Connector_JST:JST_XH_B4B-XH-AM_1x04_P2.50mm_Vertical -> Connector_JST:JST_XH_B4B-XH-A_1x04_P2.50mm_Vertical
- J15, J18, J19: footprint Connector_JST:JST_XH_B4B-XH-AM_1x04_P2.50mm_Vertical -> Connector:NS-Tech_Grove_1x04_P2mm_Vertical
- J20, J5: footprint Connector_JST:JST_XH_B2B-XH-AM_1x02_P2.50mm_Vertical -> Connector_JST:JST_XH_B2B-XH-A_1x02_P2.50mm_Vertical
- J22, J23, J24, J25, J26, J27: footprint Connector_JST:JST_XH_B3B-XH-AM_1x03_P2.50mm_Vertical -> Connector_JST:JST_XH_B3B-XH-A_1x03_P2.50mm_Vertical
- J8: footprint Footprint:4_pin_Molex -> Footprint:Molex-4Pin
- moved J1 214.1 mm to (44.2, 52.1), turned to 90 degrees
- moved C8 22.9 mm to (206.1, 60.0), turned to 90 degrees
- moved R7 18.5 mm to (74.0, 75.7), turned to 0 degrees
- moved F4 17.9 mm to (233.8, 74.1)
- moved J11 16.9 mm to (240.2, 113.2), turned to -90 degrees
- moved C7 16.0 mm to (244.2, 77.3)
- moved R8 14.5 mm to (74.0, 80.5), turned to 0 degrees
- moved R6 12.1 mm to (61.0, 81.2), turned to -90 degrees
- moved R9 11.8 mm to (74.0, 85.3), turned to 0 degrees
- moved R10 11.8 mm to (74.0, 89.7), turned to 0 degrees
- moved J8 10.0 mm to (215.6, 60.5)
- moved R25 9.79 mm to (198.9, 70.1), turned to 180 degrees
- moved R27 9.78 mm to (240.4, 124.3), turned to 180 degrees
- moved R26 9.48 mm to (184.3, 79.9), turned to 90 degrees
- moved R5 8.87 mm to (64.5, 73.6), turned to -90 degrees
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Connections:
- J10 pad 28: GND-1 -> unconnected-(J10-Pin_28-Pad28)
- U1 pad J3_1: GND-1 -> GND
Routing:
- net 3V3: track 0.00 -> 367.1 mm
- net +5V: track 38.8 -> 404.3 mm
- net IO 34: track 0.00 -> 258.6 mm
- net IO 35: track 0.00 -> 220.7 mm
- net IO 33: track 0.00 -> 203.2 mm, vias 0 -> 1
- net GPIO 21: track 0.00 -> 201.6 mm, vias 0 -> 1
- net IO 32: track 0.00 -> 189.7 mm, vias 0 -> 2
- net GPIO 2: track 36.4 -> 206.4 mm, vias 0 -> 4
- net GPIO 6: track 0.00 -> 166.4 mm, vias 0 -> 1
- net GPIO 3: track 19.4 -> 169.5 mm, vias 2 -> 5
- net IO 21: track 0.00 -> 148.0 mm
- net IO 22: track 0.00 -> 147.0 mm, vias 0 -> 2
- net IO 14: track 0.00 -> 146.5 mm, vias 0 -> 1
- net GPIO 20: track 0.00 -> 144.0 mm, vias 0 -> 4
- net IO 19: track 0.00 -> 117.7 mm
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- added copper zone on In2.Cu, net +12V
- added copper zone on In2.Cu, net /Power Distribution/12V_FUSED_MAIN
- removed copper zone on F.Cu, net +12V
- removed copper zone on B.Cu, net /Power Distribution/12V_FUSED_MAIN
- removed copper zone on F.Cu, net /Power Distribution/12V_FUSED_MAIN
Other:
- outline, holes or cut-outs redrawn
- board text added: "VertiFarm"
