File: PCB_Test.kicad_sch (KiCad schematic)
At the start: 27 parts, among them J1 Peltier, J10 Raspberry Pi 5, J13 3V3 I2C, J15 3V3 I2C, J17 3V3 I2C, J18 5V I2C, J19 3V3 I2C, J20 Switch_2, J21 Camera, J22 DS12B20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

Commit message: updated 1.0
Parts:
- added H1, H2, H3, H4: MountingHole, MountingHole:MountingHole_4mm_Pad, symbol Mechanical:MountingHole
- added J11: Peltier, TerminalBlock:TerminalBlock_Xinya_XY308-2.54-2P_1x02_P2.54mm_Horizontal, symbol Connector:Screw_Terminal_01x02
- added R27: 10k, Resistor_THT:R_Axial_DIN0207_L6.3mm_D2.5mm_P10.16mm_Horizontal, symbol Device:R
Connections:
- net GND: now also R27.2
- new net: J11.2 (Pin_2), R27.1
- new net +12V: J11.1 (Pin_1)
Other:
- moved on the sheet: J1

Commit message: version 1.0
Parts:
- removed H1, H2, H3, H4: MountingHole, MountingHole:MountingHole_4mm_Pad, symbol Mechanical:MountingHole
- added FID1, FID2, FID3, FID4: Fiducial, Fiducial:Fiducial_0.75mm_Mask1.5mm, symbol Mechanical:Fiducial
- J11: footprint TerminalBlock:TerminalBlock_Xinya_XY308-2.54-2P_1x02_P2.54mm_Horizontal -> TerminalBlock:TerminalBlock_MaiXu_MX126-5.0-02P_1x02_P5.00mm
- J13, J17, J9: footprint Connector_JST:JST_XH_B4B-XH-AM_1x04_P2.50mm_Vertical -> Connector_JST:JST_XH_B4B-XH-A_1x04_P2.50mm_Vertical
- J15, J18, J19: footprint Connector_JST:JST_XH_B4B-XH-AM_1x04_P2.50mm_Vertical -> Connector:NS-Tech_Grove_1x04_P2mm_Vertical
- J20, J5: footprint Connector_JST:JST_XH_B2B-XH-AM_1x02_P2.50mm_Vertical -> Connector_JST:JST_XH_B2B-XH-A_1x02_P2.50mm_Vertical
- J22, J23, J24, J25, J26, J27: footprint Connector_JST:JST_XH_B3B-XH-AM_1x03_P2.50mm_Vertical -> Connector_JST:JST_XH_B3B-XH-A_1x03_P2.50mm_Vertical
Connections:
- net GND-1: no longer names the net of J10.28 (Pin_28)
- no-connect marks 16 -> 17
