File: Power Distribution.kicad_sch (KiCad schematic)
At the start: 9 parts, among them J7 PCIe Header, J8 4 Pin Molex Header

Commit message: updated 1.0
Parts:
- F3: value Fuse 15A -> Fuse 30A
- J8: footprint Footprint:231834001000 -> Footprint:4_pin_Molex
Connections:
- net +12V: no longer C5.1, C6.1, D1.2 (A2), J7.10 (POWER_6), J7.9 (POWER_5)
- net 12V_FUSED_MAIN: now reaches F3.2, J7.5 (POWER_1), J7.6 (POWER_2), J7.7 (POWER_3), J7.8 (POWER_4)
- net 12V_FUSED_MAIN: now also C5.1, C6.1, D1.2 (A2), J7.10 (POWER_6), J7.9 (POWER_5)
Changed lines of the file:
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@@
+	)
+	(junction
+		(at 144.78 104.14)
+		(diameter 0)
+		(color 0 0 0 0)
 	)
 	(junction
@@
 	)
 	(junction
-		(at 144.78 104.14)
-		(diameter 0)
-		(color 0 0 0 0)
-	)
-	(junction
 		(at 102.87 72.39)
 		(diameter 0)
@@
 	(wire
 		(pts
+			(xy 102.87 68.58) (xy 102.87 72.39)
+		)
+		(stroke
+			(width 0)
+			(type default)
+		)
+	)
+	(wire
+		(pts
 			(xy 144.78 91.44) (xy 143.51 91.44)
 		)
@@
 	(wire
 		(pts
+			(xy 102.87 57.15) (xy 102.87 60.96)
+		)
+		(stroke
+			(width 0)
+			(type default)
+		)
+	)
+	(wire
+		(pts
 			(xy 144.78 96.52) (xy 143.51 96.52)
 		)
@@
 	(wire
 		(pts
-			(xy 102.87 68.58) (xy 102.87 72.39)
-		)
-		(stroke
-			(width 0)
-			(type default)
-		)
-	)
-	(wire
-		(pts
 			(xy 214.63 78.74) (xy 214.63 88.9)
 		)
@@
 	(wire
 		(pts
-			(xy 102.87 99.06) (xy 102.87 101.6)
-		)
-		(stroke
-			(width 0)
-			(type default)
-		)
-	)
-	(wire
-		(pts
 			(xy 102.87 72.39) (xy 144.78 72.39)
 		)
@@
 	(wire
 		(pts
+			(xy 102.87 72.39) (xy 102.87 99.06)
+		)
+		(stroke
+			(width 0)
+			(type default)
+		)
+	)
+	(wire
+		(pts
 			(xy 144.78 104.14) (xy 143.51 104.14)
 		)
@@
 	(wire
 		(pts
-			(xy 102.87 72.39) (xy 102.87 76.2)
-		)
-		(stroke
-			(width 0)
-			(type default)
-		)
-	)
-	(wire
-		(pts
 			(xy 190.5 106.68) (xy 190.5 109.22)
 		)
@@
 	(wire
 		(pts
-			(xy 102.87 101.6) (xy 102.87 104.14)
+			(xy 102.87 99.06) (xy 102.87 104.14)
 		)
 		(stroke
@@
 	(wire
 		(pts
-			(xy 102.87 83.82) (xy 102.87 99.06)
-		)
-		(stroke
-			(width 0)
-			(type default)
-		)
-	)
-	(wire
-		(pts
 			(xy 236.22 91.44) (xy 236.22 95.25)
 		)
@@
 			(width 0)
 			(type default)
+		)
+	)
+	(label "12V_RAW"
+		(at 102.87 59.69 0)
+		(effects
+			(font
+				(size 1.27 1.27)
+			)
+			(justify left bottom)
+		)
+	)
+	(label "12V_FUSED_MAIN"
+		(at 102.87 81.28 180)
+		(effects
+			(font
+				(size 1.27 1.27)
+			)
+			(justify right bottom)
 		)
 	)
@@
 			)
 		)
-		(property "Footprint" "Footprint:231834001000"
+		(property "Footprint" "Footprint:4_pin_Molex"
 			(at 209.55 183.82 0)
 			(hide yes)
@@
 	)
 	(symbol
+		(lib_id "Device:Fuse")
+		(at 102.87 64.77 0)
+		(unit 1)
+		(body_style 1)
+		(exclude_from_sim no)
+		(in_bom yes)
+		(on_board yes)
+		(in_pos_files yes)
+		(dnp no)
+		(fields_autoplaced yes)
+		(property "Reference" "F3"
+			(at 105.41 63.4999 0)
+			(show_name no)
+			(do_not_autoplace no)
+			(effects
+				(font
+					(size 1.27 1.27)
+				)
+				(justify left)
+			)
+		)
+		(property "Value" "Fuse 30A"
+			(at 105.41 66.0399 0)
+			(show_name no)
+			(do_not_autoplace no)
+			(effects
+				(font
+					(size 1.27 1.27)
+				)
+				(justify left)
+			)
+		)
+		(property "Footprint" "Fuse:Fuse_Blade_ATO_directSolder"
+			(at 101.092 64.77 90)
+			(hide yes)
+			(show_name no)
+			(do_not_autoplace no)
+			(effects
+				(font
+					(size 1.27 1.27)
+				)
+			)
+		)
+		(property "Datasheet" ""
+			(at 102.87 64.77 0)
+			(hide yes)
+			(show_name no)
+			(do_not_autoplace no)
+			(effects
+				(font
+					(size 1.27 1.27)
+				)
+			)
+		)
+		(property "Description" "Fuse"
+			(at 102.87 64.77 0)
+			(hide yes)
+			(show_name no)
+			(do_not_autoplace no)
+			(effects
+				(font
+					(size 1.27 1.27)
+				)
+			)
+		)
+		(pin "1"
+		)
+		(pin "2"
+		)
+		(instances
+			(project "PCB_Test"
+				(path "/af4f5558-672d-42f1-bcb2-d73fc89abcc2/e0a23ab8-28f9-4c3b-ac56-8ad0faecca7e"
+					(reference "F3")
+					(unit 1)
+				)
+			)
+		)
+	)
+	(symbol
 		(lib_id "power:+5V")
 		(at 226.06 86.36 0)
@@
 	(symbol
 		(lib_id "power:+12V")
-		(at 102.87 68.58 0)
+		(at 102.87 57.15 0)
 		(unit 1)
 		(body_style 1)
@@
 		(fields_autoplaced yes)
 		(property "Reference" "#PWR034"
-			(at 102.87 72.39 0)
+			(at 102.87 60.96 0)
 			(hide yes)
 			(show_name no)
@@
 		)
 		(property "Value" "+12V"
-			(at 102.87 63.5 0)
+			(at 102.87 52.07 0)
 			(show_name no)
 			(do_not_autoplace no)
@@
 		)
 		(property "Footprint" ""
-			(at 102.87 68.58 0)
+			(at 102.87 57.15 0)
 			(hide yes)
 			(show_name no)
@@
 		)
 		(property "Datasheet" ""
-			(at 102.87 68.58 0)
+			(at 102.87 57.15 0)
 			(hide yes)
 			(show_name no)
@@
 		)
 		(property "Description" "Power symbol creates a global label with name \"+12V\""
-			(at 102.87 68.58 0)
+			(at 102.87 57.15 0)
 			(hide yes)
 			(show_name no)
@@
 					(unit 1)
 				)
-			)
-		)
-	)
-	(symbol
-		(lib_id "Device:Fuse")
-		(at 102.87 80.01 0)
-		(unit 1)
-		(body_style 1)
-		(exclude_from_sim no)
-		(in_bom yes)
-		(on_board yes)
-		(in_pos_files yes)
-		(dnp no)
-		(fields_autoplaced yes)
-		(property "Reference" "F3"
-			(at 105.41 78.7399 0)
-			(show_name no)
-			(do_not_autoplace no)
-			(effects
-				(font
-					(size 1.27 1.27)
-				)
-				(justify left)
-			)
-		)
-		(property "Value" "Fuse 15A"
-			(at 105.41 81.2799 0)
-			(show_name no)
-			(do_not_autoplace no)
-			(effects
-				(font
-					(size 1.27 1.27)
-				)
-				(justify left)
-			)
-		)
-		(property "Footprint" "Fuse:Fuse_Blade_ATO_directSolder"
-			(at 101.092 80.01 90)
-			(hide yes)
-			(show_name no)
-			(do_not_autoplace no)
-			(effects
-				(font
-					(size 1.27 1.27)
-				)
-			)
-		)
-		(property "Datasheet" ""
-			(at 102.87 80.01 0)
-			(hide yes)
-			(show_name no)
-			(do_not_autoplace no)
-			(effects
-				(font
-					(size 1.27 1.27)
-				)
-			)
-		)
-		(property "Description" "Fuse"
-			(at 102.87 80.01 0)
-			(hide yes)
-			(show_name no)
-			(do_not_autoplace no)
-			(effects
-				(font
-					(size 1.27 1.27)
-				)
-			)
-		)
-		(pin "1"
-		)
-		(pin "2"
-		)
-		(instances
-			(project "PCB_Test"
-				(path "/af4f5558-672d-42f1-bcb2-d73fc89abcc2/e0a23ab8-28f9-4c3b-ac56-8ad0faecca7e"
-					(reference "F3")
-					(unit 1)
-				)

Commit message: Describe the task you completed
Connections:
- net +12V: now also C5.1, C6.1, D1.2 (A2)
- net 12V_FUSED_MAIN: no longer C5.1, C6.1, D1.2 (A2)
Changed lines of the file:
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@@
+	)
+	(junction
+		(at 83.82 72.39)
+		(diameter 0)
+		(color 0 0 0 0)
+	)
+	(junction
+		(at 144.78 104.14)
+		(diameter 0)
+		(color 0 0 0 0)
+	)
+	(junction
+		(at 100.33 63.5)
+		(diameter 0)
+		(color 0 0 0 0)
+	)
+	(junction
+		(at 100.33 99.06)
+		(diameter 0)
+		(color 0 0 0 0)
 	)
 	(junction
@@
 	)
 	(junction
-		(at 144.78 104.14)
-		(diameter 0)
-		(color 0 0 0 0)
-	)
-	(junction
-		(at 102.87 99.06)
-		(diameter 0)
-		(color 0 0 0 0)
-	)
-	(junction
-		(at 102.87 72.39)
-		(diameter 0)
-		(color 0 0 0 0)
-	)
-	(junction
-		(at 83.82 72.39)
-		(diameter 0)
-		(color 0 0 0 0)
-	)
-	(junction
 		(at 190.5 106.68)
 		(diameter 0)
@@
 	)
 	(junction
+		(at 100.33 104.14)
+		(diameter 0)
+		(color 0 0 0 0)
+	)
+	(junction
 		(at 144.78 99.06)
 		(diameter 0)
@@
 	)
 	(junction
+		(at 100.33 80.01)
+		(diameter 0)
+		(color 0 0 0 0)
+	)
+	(junction
 		(at 144.78 106.68)
 		(diameter 0)
@@
 	)
 	(junction
-		(at 102.87 101.6)
+		(at 100.33 101.6)
 		(diameter 0)
 		(color 0 0 0 0)
@@
 	(junction
 		(at 144.78 111.76)
-		(diameter 0)
-		(color 0 0 0 0)
-	)
-	(junction
-		(at 102.87 104.14)
 		(diameter 0)
 		(color 0 0 0 0)
@@
 	(wire
 		(pts
-			(xy 102.87 68.58) (xy 102.87 72.39)
-		)
-		(stroke
-			(width 0)
-			(type default)
-		)
-	)
-	(wire
-		(pts
 			(xy 144.78 91.44) (xy 143.51 91.44)
 		)
@@
 	(wire
 		(pts
-			(xy 102.87 101.6) (xy 105.41 101.6)
-		)
-		(stroke
-			(width 0)
-			(type default)
-		)
-	)
-	(wire
-		(pts
 			(xy 83.82 101.6) (xy 83.82 95.25)
 		)
@@
 	(wire
 		(pts
-			(xy 102.87 57.15) (xy 102.87 60.96)
+			(xy 100.33 57.15) (xy 100.33 63.5)
 		)
 		(stroke
@@
 	(wire
 		(pts
+			(xy 100.33 63.5) (xy 83.82 63.5)
+		)
+		(stroke
+			(width 0)
+			(type default)
+		)
+	)
+	(wire
+		(pts
 			(xy 104.14 91.44) (xy 104.14 93.98)
 		)
@@
 	(wire
 		(pts
+			(xy 100.33 80.01) (xy 144.78 80.01)
+		)
+		(stroke
+			(width 0)
+			(type default)
+		)
+	)
+	(wire
+		(pts
 			(xy 248.92 95.25) (xy 248.92 91.44)
 		)
@@
 	(wire
 		(pts
+			(xy 100.33 73.66) (xy 100.33 80.01)
+		)
+		(stroke
+			(width 0)
+			(type default)
+		)
+	)
+	(wire
+		(pts
+			(xy 100.33 80.01) (xy 100.33 99.06)
+		)
+		(stroke
+			(width 0)
+			(type default)
+		)
+	)
+	(wire
+		(pts
 			(xy 190.5 91.44) (xy 190.5 106.68)
 		)
@@
 	(wire
 		(pts
-			(xy 102.87 72.39) (xy 144.78 72.39)
-		)
-		(stroke
-			(width 0)
-			(type default)
-		)
-	)
-	(wire
-		(pts
 			(xy 248.92 102.87) (xy 248.92 106.68)
 		)
@@
 	(wire
 		(pts
-			(xy 144.78 72.39) (xy 144.78 88.9)
-		)
-		(stroke
-			(width 0)
-			(type default)
-		)
-	)
-	(wire
-		(pts
-			(xy 102.87 72.39) (xy 102.87 99.06)
-		)
-		(stroke
-			(width 0)
-			(type default)
-		)
-	)
-	(wire
-		(pts
 			(xy 144.78 104.14) (xy 143.51 104.14)
 		)
@@
 	(wire
 		(pts
+			(xy 100.33 101.6) (xy 100.33 104.14)
+		)
+		(stroke
+			(width 0)
+			(type default)
+		)
+	)
+	(wire
+		(pts
 			(xy 144.78 99.06) (xy 144.78 101.6)
 		)
@@
 	(wire
 		(pts
+			(xy 83.82 63.5) (xy 83.82 72.39)
+		)
+		(stroke
+			(width 0)
+			(type default)
+		)
+	)
+	(wire
+		(pts
 			(xy 190.5 106.68) (xy 190.5 109.22)
 		)
@@
 	(wire
 		(pts
-			(xy 83.82 72.39) (xy 102.87 72.39)
+			(xy 100.33 104.14) (xy 100.33 106.68)
 		)
 		(stroke
@@
 	(wire
 		(pts
+			(xy 100.33 99.06) (xy 105.41 99.06)
+		)
+		(stroke
+			(width 0)
+			(type default)
+		)
+	)
+	(wire
+		(pts
 			(xy 63.5 111.76) (xy 144.78 111.76)
 		)
@@
 	(wire
 		(pts
-			(xy 102.87 99.06) (xy 102.87 104.14)
+			(xy 100.33 99.06) (xy 100.33 101.6)
+		)
+		(stroke
+			(width 0)
+			(type default)
+		)
+	)
+	(wire
+		(pts
+			(xy 144.78 88.9) (xy 144.78 80.01)
 		)
 		(stroke
@@
 	(wire
 		(pts
-			(xy 102.87 106.68) (xy 105.41 106.68)
-		)
-		(stroke
-			(width 0)
-			(type default)
-		)
-	)
-	(wire
-		(pts
 			(xy 63.5 101.6) (xy 83.82 101.6)
 		)
@@
 	(wire
 		(pts
-			(xy 102.87 104.14) (xy 102.87 106.68)
+			(xy 100.33 101.6) (xy 105.41 101.6)
 		)
 		(stroke
@@
 	(wire
 		(pts
+			(xy 100.33 104.14) (xy 105.41 104.14)
+		)
+		(stroke
+			(width 0)
+			(type default)
+		)
+	)
+	(wire
+		(pts
+			(xy 100.33 106.68) (xy 105.41 106.68)
+		)
+		(stroke
+			(width 0)
+			(type default)
+		)
+	)
+	(wire
+		(pts
 			(xy 105.41 91.44) (xy 104.14 91.44)
 		)
@@
 	(wire
 		(pts
-			(xy 102.87 104.14) (xy 105.41 104.14)
+			(xy 100.33 63.5) (xy 100.33 66.04)
 		)
 		(stroke
@@
 		)
 	)
-	(wire
-		(pts
-			(xy 105.41 99.06) (xy 102.87 99.06)
-		)
-		(stroke
-			(width 0)
-			(type default)
-		)
-	)
 	(label "12V_RAW"
-		(at 102.87 59.69 0)
+		(at 100.33 58.42 0)
 		(effects
 			(font
@@
 	)
 	(label "12V_FUSED_MAIN"
-		(at 102.87 81.28 180)
+		(at 100.33 76.2 0)
 		(effects
 			(font
 				(size 1.27 1.27)
 			)
-			(justify right bottom)
+			(justify left bottom)
 		)
 	)
@@
 	(symbol
 		(lib_id "Device:Fuse")
-		(at 102.87 64.77 0)
+		(at 100.33 69.85 0)
 		(unit 1)
 		(body_style 1)
@@
 		(fields_autoplaced yes)
 		(property "Reference" "F3"
-			(at 105.41 63.4999 0)
+			(at 102.87 68.5799 0)
 			(show_name no)
 			(do_not_autoplace no)
@@
 		)
 		(property "Value" "Fuse 30A"
-			(at 105.41 66.0399 0)
+			(at 102.87 71.1199 0)
 			(show_name no)
 			(do_not_autoplace no)
@@
 		)
 		(property "Footprint" "Fuse:Fuse_Blade_ATO_directSolder"
-			(at 101.092 64.77 90)
+			(at 98.552 69.85 90)
 			(hide yes)
 			(show_name no)
@@
 		)
 		(property "Datasheet" ""
-			(at 102.87 64.77 0)
+			(at 100.33 69.85 0)
 			(hide yes)
 			(show_name no)
@@
 		)
 		(property "Description" "Fuse"
-			(at 102.87 64.77 0)
+			(at 100.33 69.85 0)
 			(hide yes)
 			(show_name no)
@@
 	(symbol
 		(lib_id "power:+12V")
-		(at 102.87 57.15 0)
+		(at 100.33 57.15 0)
 		(unit 1)
 		(body_style 1)
@@
 		(fields_autoplaced yes)
 		(property "Reference" "#PWR034"
-			(at 102.87 60.96 0)
+			(at 100.33 60.96 0)
 			(hide yes)
 			(show_name no)
@@
 		)
 		(property "Value" "+12V"
-			(at 102.87 52.07 0)
+			(at 100.33 52.07 0)
 			(show_name no)
 			(do_not_autoplace no)
@@
 		)
 		(property "Footprint" ""
-			(at 102.87 57.15 0)
+			(at 100.33 57.15 0)
 			(hide yes)
 			(show_name no)
@@
 		)
 		(property "Datasheet" ""
-			(at 102.87 57.15 0)
+			(at 100.33 57.15 0)
 			(hide yes)
 			(show_name no)
@@
 		)
 		(property "Description" "Power symbol creates a global label with name \"+12V\""
-			(at 102.87 57.15 0)
-			(hide yes)
-			(show_name no)
+			(at 100.33 57.15 0)
+			(hide yes)
+			(show_name no)

Commit message: version 1.0
Parts:
- F4: value Fuse 2A -> Fuse 11A; footprint Fuse:Fuse_Blade_ATO_directSolder -> Fuse:Fuseholder_Cylinder-5x20mm_Schurter_0031_8201_Horizontal_Open
- J8: footprint Footprint:4_pin_Molex -> Footprint:Molex-4Pin
Changed lines of the file:
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@@
 			)
 		)
-		(property "Footprint" "Footprint:4_pin_Molex"
+		(property "Footprint" "Footprint:Molex-4Pin"
 			(at 209.55 183.82 0)
 			(hide yes)
@@
 			)
 		)
-		(property "Value" "Fuse 2A"
+		(property "Value" "Fuse 11A"
 			(at 219.71 87.63 90)
 			(show_name no)
@@
 			)
 		)
-		(property "Footprint" "Fuse:Fuse_Blade_ATO_directSolder"
+		(property "Footprint" "Fuse:Fuseholder_Cylinder-5x20mm_Schurter_0031_8201_Horizontal_Open"
 			(at 219.71 93.218 90)
-			(hide yes)
-			(show_name no)
-			(do_not_autoplace no)
+			(show_name no)
+			(do_not_autoplace no)
