File: Power Distribution.kicad_sch (KiCad schematic)
At the start: 9 parts, among them J7 PCIe Header, J8 4 Pin Molex Header

Commit message: Version 2.0
Parts:
- F3: value Fuse 30A -> Fuse 40A; footprint Fuse:Fuse_Blade_ATO_directSolder -> Fuse_Blade:Fuse_Blade_ATO_directSolder_32V_40A
- F4: value Fuse 11A -> Fuse 10A; footprint Fuse:Fuseholder_Cylinder-5x20mm_Schurter_0031_8201_Horizontal_Open -> Fuse_Blade:Fuse_Blade_ATO_12VDC_10A
Changed lines of the file:
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@@
 		)
 		(instances
-			(project "PCB_Test"
+			(project "VertiFarm_PCB"
 				(path "/af4f5558-672d-42f1-bcb2-d73fc89abcc2/e0a23ab8-28f9-4c3b-ac56-8ad0faecca7e"
 					(reference "J8")
@@
 		)
 		(instances
-			(project "PCB_Test"
+			(project "VertiFarm_PCB"
 				(path "/af4f5558-672d-42f1-bcb2-d73fc89abcc2/e0a23ab8-28f9-4c3b-ac56-8ad0faecca7e"
 					(reference "#PWR036")
@@
 		)
 		(instances
-			(project "PCB_Test"
+			(project "VertiFarm_PCB"
 				(path "/af4f5558-672d-42f1-bcb2-d73fc89abcc2/e0a23ab8-28f9-4c3b-ac56-8ad0faecca7e"
 					(reference "C7")
@@
 			)
 		)
-		(property "Value" "Fuse 30A"
+		(property "Value" "Fuse 40A"
 			(at 102.87 71.1199 0)
 			(show_name no)
@@
 			)
 		)
-		(property "Footprint" "Fuse:Fuse_Blade_ATO_directSolder"
+		(property "Footprint" "Fuse_Blade:Fuse_Blade_ATO_directSolder_32V_40A"
 			(at 98.552 69.85 90)
 			(hide yes)
@@
 		)
 		(instances
-			(project "PCB_Test"
+			(project "VertiFarm_PCB"
 				(path "/af4f5558-672d-42f1-bcb2-d73fc89abcc2/e0a23ab8-28f9-4c3b-ac56-8ad0faecca7e"
 					(reference "F3")
@@
 		)
 		(instances
-			(project "PCB_Test"
+			(project "VertiFarm_PCB"
 				(path "/af4f5558-672d-42f1-bcb2-d73fc89abcc2/e0a23ab8-28f9-4c3b-ac56-8ad0faecca7e"
 					(reference "#PWR037")
@@
 		)
 		(instances
-			(project "PCB_Test"
+			(project "VertiFarm_PCB"
 				(path "/af4f5558-672d-42f1-bcb2-d73fc89abcc2/e0a23ab8-28f9-4c3b-ac56-8ad0faecca7e"
 					(reference "C5")
@@
 		)
 		(instances
-			(project "PCB_Test"
+			(project "VertiFarm_PCB"
 				(path "/af4f5558-672d-42f1-bcb2-d73fc89abcc2/e0a23ab8-28f9-4c3b-ac56-8ad0faecca7e"
 					(reference "C8")
@@
 			)
 		)
-		(property "Value" "Fuse 11A"
+		(property "Value" "Fuse 10A"
 			(at 219.71 87.63 90)
 			(show_name no)
@@
 			)
 		)
-		(property "Footprint" "Fuse:Fuseholder_Cylinder-5x20mm_Schurter_0031_8201_Horizontal_Open"
+		(property "Footprint" "Fuse_Blade:Fuse_Blade_ATO_12VDC_10A"
 			(at 219.71 93.218 90)
+			(hide yes)
 			(show_name no)
 			(do_not_autoplace no)
@@
 		)
 		(instances
-			(project "PCB_Test"
+			(project "VertiFarm_PCB"
 				(path "/af4f5558-672d-42f1-bcb2-d73fc89abcc2/e0a23ab8-28f9-4c3b-ac56-8ad0faecca7e"
 					(reference "F4")
@@
 		)
 		(instances
-			(project "PCB_Test"
+			(project "VertiFarm_PCB"
 				(path "/af4f5558-672d-42f1-bcb2-d73fc89abcc2/e0a23ab8-28f9-4c3b-ac56-8ad0faecca7e"
 					(reference "#PWR034")
@@
 		)
 		(instances
-			(project "PCB_Test"
+			(project "VertiFarm_PCB"
 				(path "/af4f5558-672d-42f1-bcb2-d73fc89abcc2/e0a23ab8-28f9-4c3b-ac56-8ad0faecca7e"
 					(reference "D1")
@@
 		)
 		(instances
-			(project "PCB_Test"
+			(project "VertiFarm_PCB"
 				(path "/af4f5558-672d-42f1-bcb2-d73fc89abcc2/e0a23ab8-28f9-4c3b-ac56-8ad0faecca7e"
 					(reference "J7")
@@
 		)
 		(instances
-			(project "PCB_Test"
+			(project "VertiFarm_PCB"
 				(path "/af4f5558-672d-42f1-bcb2-d73fc89abcc2/e0a23ab8-28f9-4c3b-ac56-8ad0faecca7e"
 					(reference "#PWR035")
@@
 		)
 		(instances
-			(project "PCB_Test"
+			(project "VertiFarm_PCB"
 				(path "/af4f5558-672d-42f1-bcb2-d73fc89abcc2/e0a23ab8-28f9-4c3b-ac56-8ad0faecca7e"
 					(reference "C6")

Commit message: Updated the Fuses Footprints and Corrected Layout
Parts:
- F3: footprint Fuse_Blade:Fuse_Blade_ATO_directSolder_32V_40A -> Footprint:Fuse_Blade_ATO_directSolder_32V_40A
- F4: footprint Fuse_Blade:Fuse_Blade_ATO_12VDC_10A -> Footprint:Fuse_Blade_ATO_12VDC_10A
Changed lines of the file:
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@@
 			)
 		)
-		(property "Footprint" "Fuse_Blade:Fuse_Blade_ATO_directSolder_32V_40A"
+		(property "Footprint" "Footprint:Fuse_Blade_ATO_directSolder_32V_40A"
 			(at 98.552 69.85 90)
-			(hide yes)
 			(show_name no)
 			(do_not_autoplace no)
@@
 			)
 		)
-		(property "Footprint" "Fuse_Blade:Fuse_Blade_ATO_12VDC_10A"
+		(property "Footprint" "Footprint:Fuse_Blade_ATO_12VDC_10A"
 			(at 219.71 93.218 90)
 			(hide yes)

Commit message: updated the connector pins
Changed lines of the file:
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@@
 		(property "Footprint" "Footprint:Fuse_Blade_ATO_directSolder_32V_40A"
 			(at 98.552 69.85 90)
+			(hide yes)
 			(show_name no)
 			(do_not_autoplace no)
